File: kicad/reflowmaster2000plus.sch (KiCad schematic (older format))
At the start: 20 parts, among them IC1 TLP3036, U1 TRIAC, U2 TLC2272

Commit message: [mod] updated schema&pcb
Parts:
- removed D4: SCHOTTKY, ~, symbol SCHOTTKY
- removed R3: R, ~, symbol R
- removed RV2: POT, ~, symbol POT
- added D4: VREFDIODE, ~, symbol VREFDIODE
- added P1: CONN_8, symbol CONN_8
- added P2: Toaster, symbol CONN_2
- added P3: 220V, symbol CONN_2
- D2: value ZENER -> BAT46
- D3: value SCHOTTKY -> BZX55C5V1
Connections:
- net labels added: +12V, AGND, KTYa, KTYc, PGND, PWRctrl, SGND, Uclamp
- net labels removed: 1, 4, I0, input, vref
- wire segments 34 -> 42
Other:
- moved on the sheet: C1, C2, C3, D1, D2, D3, IC1, R1, R2, R4, R5, R6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
